File: PCB.kicad_pcb (KiCad board)
At the start: 4 copper layers, 42 parts, among them J1 USB_C_Receptacle_USB2.0, J2 JST - 1.00mm 4 Pin, SW1 MX_SW_solder, SW2 MX_SW_solder, SW3 MX_SW_solder, SW4 MX_SW_solder, SW72 SW_Push, SW73 SW_Push, U1 RP2040, U2 SOP-8 SPI FLASH, U3 USBLC6-2SC6, U4 3.3V Fixed Regulator, Y1 12MHz Crystal 3225

Commit message: Layout complete
Parts:
- removed C1, C2: 30p, Capacitor_SMD:C_0402_1005Metric
- removed C10, C12, C13, C15, C3: 1u, Capacitor_SMD:C_0402_1005Metric
- removed C11, C14, C16, C4, C5, C6, C7, C8, C9: 100n, Capacitor_SMD:C_0402_1005Metric
- removed D65: LED, marbastlib-mx:LED_MX_3mm
- removed F1: 700mA, Fuse:Fuse_0402_1005Metric
- removed FB1: 100 Ohm @ 100 MHz, Inductor_SMD:L_0402_1005Metric
- removed J2: JST - 1.00mm 4 Pin, Connector_JST:JST_SH_SM04B-SRSS-TB_1x04-1MP_P1.00mm_Horizontal
- removed R1, R2: 22, Resistor_SMD:R_0402_1005Metric
- removed R3: 1k, Resistor_SMD:R_0402_1005Metric
- removed R4: 5.1k, Resistor_SMD:R_0402_1005Metric
- removed R7: R_Small_US, Resistor_SMD:R_0402_1005Metric
- removed SW72, SW73: SW_Push, Button_Switch_SMD:SW_SPST_SKQG_WithoutStem
- removed U1: RP2040, Package_DFN_QFN:QFN-56-1EP_7x7mm_P0.4mm_EP3.2x3.2mm_ThermalVias
- removed U3: USBLC6-2SC6, Package_TO_SOT_SMD:SOT-23-6
- removed U4: 3.3V Fixed Regulator, Package_TO_SOT_SMD:TSOT-23
- removed Y1: 12MHz Crystal 3225, Crystal:Crystal_SMD_3225-4Pin_3.2x2.5mm
- added C17: 1u, Capacitor_SMD:C_0402_1005Metric, B.Cu at (25.3, 31.1)
- added C18: 1u, Capacitor_SMD:C_0402_1005Metric, B.Cu at (25.3, 33.1)
- added C19: 4.7u, Capacitor_SMD:C_0402_1005Metric, B.Cu at (62.8, 65.9)
- added C20: 100n, Capacitor_SMD:C_0402_1005Metric, B.Cu at (64.4, 73.8)
- added C21: 100n, Capacitor_SMD:C_0402_1005Metric, B.Cu at (70.8, 64.4)
- added C22: 100n, Capacitor_SMD:C_0402_1005Metric, B.Cu at (72.4, 70.6)
- added C23: 100n, Capacitor_SMD:C_0402_1005Metric, B.Cu at (61.8, 65.9)
- added D10: D_Small, Diode_SMD:D_SOD-123, B.Cu at (218.8, 41.7)
- added D11: D_Small, Diode_SMD:D_SOD-123, B.Cu at (237.8, 41.7)
- added D12: D_Small, Diode_SMD:D_SOD-123, B.Cu at (256.9, 41.7)
- added D13: D_Small, Diode_SMD:D_SOD-123, B.Cu at (49.7, 60.7)
- added D14: D_Small, Diode_SMD:D_SOD-123, B.Cu at (71.1, 60.7)
- added D15: D_Small, Diode_SMD:D_SOD-123, B.Cu at (90.2, 60.7)
- added D16: D_Small, Diode_SMD:D_SOD-123, B.Cu at (109.2, 60.7)
- added D17: D_Small, Diode_SMD:D_SOD-123, B.Cu at (128.3, 60.7)
- added D18: D_Small, Diode_SMD:D_SOD-123, B.Cu at (147.3, 60.7)
- added D19: D_Small, Diode_SMD:D_SOD-123, B.Cu at (166.4, 60.7)
- added D20: D_Small, Diode_SMD:D_SOD-123, B.Cu at (185.4, 60.7)
- added D21: D_Small, Diode_SMD:D_SOD-123, B.Cu at (204.5, 60.7)
- added D22: D_Small, Diode_SMD:D_SOD-123, B.Cu at (223.5, 60.7)
- added D23: D_Small, Diode_SMD:D_SOD-123, B.Cu at (249.7, 60.7)
- added D24: D_Small, Diode_SMD:D_SOD-123, B.Cu at (54.5, 79.8)
- added D25: D_Small, Diode_SMD:D_SOD-123, B.Cu at (80.6, 79.8)
- added D26: D_Small, Diode_SMD:D_SOD-123, B.Cu at (99.7, 79.8)
- added D27: D_Small, Diode_SMD:D_SOD-123, B.Cu at (118.7, 79.8)
- added D28: D_Small, Diode_SMD:D_SOD-123, B.Cu at (137.8, 79.8)
- added D29: D_Small, Diode_SMD:D_SOD-123, B.Cu at (156.8, 79.8)
- added D30: D_Small, Diode_SMD:D_SOD-123, B.Cu at (175.9, 79.8)
- added D31: D_Small, Diode_SMD:D_SOD-123, B.Cu at (194.9, 79.8)
- added D32: D_Small, Diode_SMD:D_SOD-123, B.Cu at (214.0, 79.8)
- added D33: D_Small, Diode_SMD:D_SOD-123, B.Cu at (233.0, 79.8)
- added D34: D_Small, Diode_SMD:D_SOD-123, B.Cu at (254.5, 79.8)
- added D35: D_Small, Diode_SMD:D_SOD-123, B.Cu at (49.7, 98.8)
- added D36: D_Small, Diode_SMD:D_SOD-123, B.Cu at (71.1, 98.8)
- added D37: D_Small, Diode_SMD:D_SOD-123, B.Cu at (92.6, 98.8)
- added D38: D_Small, Diode_SMD:D_SOD-123, B.Cu at (130.7, 98.8)
- added D39: D_Small, Diode_SMD:D_SOD-123, B.Cu at (178.3, 98.8)
- added D40: D_Small, Diode_SMD:D_SOD-123, B.Cu at (211.6, 98.8)
- added D41: D_Small, Diode_SMD:D_SOD-123, B.Cu at (233.0, 98.8)
- added D42: D_Small, Diode_SMD:D_SOD-123, B.Cu at (243.3, 99.6)
- added D44: D_Small, Diode_SMD:D_SOD-123, B.Cu at (257.0, 98.4)
- added D45: LED, Resistor_SMD:R_0603_1608Metric, B.Cu at (12.3, 40.7)
- added D5: D_Small, Diode_SMD:D_SOD-123, B.Cu at (123.5, 41.7)
- added D6: D_Small, Diode_SMD:D_SOD-123, B.Cu at (142.6, 41.7)
- added D7: D_Small, Diode_SMD:D_SOD-123, B.Cu at (161.6, 41.7)
- added D8: D_Small, Diode_SMD:D_SOD-123, B.Cu at (180.7, 41.7)
- added D9: D_Small, Diode_SMD:D_SOD-123, B.Cu at (199.7, 41.7)
- added J4: TC2030_SWD, PCM_marbastlib-various:CON_TC2030_outlined, B.Cu at (10.5, 32.7)
- added Q2: PMOS, Package_TO_SOT_SMD:SOT-323_SC-70, B.Cu at (247.8, 39.4)
- added Q3: PMOS, Package_TO_SOT_SMD:SOT-323_SC-70, B.Cu at (40.8, 41.4)
- added Q4: PMOS, Package_TO_SOT_SMD:SOT-323_SC-70, B.Cu at (12.3, 37.0)
- added R6: 100k, Resistor_SMD:R_0402_1005Metric, B.Cu at (247.8, 37.4)
- added R8: 470, Resistor_SMD:R_0603_1608Metric, B.Cu at (12.3, 43.2)
- added S1: MX_stab, marbastlib-mx:STAB_MX_P_7u, F.Cu at (152.1, 94.1)
- added S2: MX_stab, marbastlib-mx:STAB_MX_P_10u, F.Cu at (152.1, 94.1)
- added S3: MX_stab, marbastlib-mx:STAB_MX_P_3u, F.Cu at (180.7, 94.1)
- added S35: MX_stab, marbastlib-mx:STAB_MX_P_2.25u, F.Cu at (245.0, 75.0)
- added S4: MX_stab, marbastlib-mx:STAB_MX_P_2.25u, F.Cu at (178.3, 94.1)
- added S40: MX_stab, marbastlib-mx:STAB_MX_P_3u, F.Cu at (123.5, 94.1)
- added S41: MX_stab, marbastlib-mx:STAB_MX_P_2.75u, F.Cu at (130.7, 94.1)
- added SW10: MX_SW_solder, marbastlib-mx:SW_MX_1u, F.Cu at (218.8, 36.9)
- added SW11: MX_SW_solder, marbastlib-mx:SW_MX_1u, F.Cu at (237.8, 36.9)
- added SW12: MX_SW_solder, marbastlib-mx:SW_MX_1u, F.Cu at (256.9, 36.9)
- added SW13: MX_SW_solder, marbastlib-mx:SW_MX_1.25u, F.Cu at (49.7, 56.0)
- added SW14: MX_SW_solder, marbastlib-mx:SW_MX_1u, F.Cu at (71.1, 56.0)
- added SW15: MX_SW_solder, marbastlib-mx:SW_MX_1u, F.Cu at (90.2, 56.0)
- added SW16: MX_SW_solder, marbastlib-mx:SW_MX_1u, F.Cu at (109.2, 56.0)
- added SW17: MX_SW_solder, marbastlib-mx:SW_MX_1u, F.Cu at (128.3, 56.0)
- added SW18: MX_SW_solder, marbastlib-mx:SW_MX_1u, F.Cu at (147.3, 56.0)
- added SW19: MX_SW_solder, marbastlib-mx:SW_MX_1u, F.Cu at (166.4, 56.0)
- added SW20: MX_SW_solder, marbastlib-mx:SW_MX_1u, F.Cu at (185.4, 56.0)
- added SW21: MX_SW_solder, marbastlib-mx:SW_MX_1u, F.Cu at (204.5, 56.0)
- added SW22: MX_SW_solder, marbastlib-mx:SW_MX_1u, F.Cu at (223.5, 56.0)
- added SW23: MX_SW_solder, marbastlib-mx:SW_MX_1.75u, F.Cu at (249.7, 56.0)
- added SW24: MX_SW_solder, marbastlib-mx:SW_MX_1.75u, F.Cu at (54.5, 75.0)
- added SW25: MX_SW_solder, marbastlib-mx:SW_MX_1u, F.Cu at (80.6, 75.0)
- added SW26: MX_SW_solder, marbastlib-mx:SW_MX_1u, F.Cu at (99.7, 75.0)
- added SW27: MX_SW_solder, marbastlib-mx:SW_MX_1u, F.Cu at (118.7, 75.0)
- added SW28: MX_SW_solder, marbastlib-mx:SW_MX_1u, F.Cu at (137.8, 75.0)
- added SW29: MX_SW_solder, marbastlib-mx:SW_MX_1u, F.Cu at (156.8, 75.0)
- added SW30: MX_SW_solder, marbastlib-mx:SW_MX_1u, F.Cu at (175.9, 75.0)
- added SW31: MX_SW_solder, marbastlib-mx:SW_MX_1u, F.Cu at (194.9, 75.0)
- added SW32: MX_SW_solder, marbastlib-mx:SW_MX_1u, F.Cu at (214.0, 75.0)
- added SW33: MX_SW_solder, marbastlib-mx:SW_MX_1u, F.Cu at (233.0, 75.0)
- added SW34: MX_SW_solder, marbastlib-mx:SW_MX_1.25u, F.Cu at (254.5, 75.0)
- added SW35: MX_SW_solder, marbastlib-mx:SW_MX_1u, F.Cu at (47.3, 94.1)
- added SW36: MX_SW_solder, marbastlib-mx:SW_MX_1u, F.Cu at (66.4, 94.1)
- added SW37: MX_SW_solder, marbastlib-mx:SW_MX_1.5u, F.Cu at (71.1, 94.1)
- added SW38: MX_SW_solder, marbastlib-mx:SW_MX_1u, F.Cu at (85.4, 94.1)
- added SW39: MX_SW_solder, marbastlib-mx:SW_MX_1u, F.Cu at (94.9, 94.1)
- added SW40: MX_SW_solder, marbastlib-mx:SW_MX_1u, F.Cu at (123.5, 94.1)
- added SW41: MX_SW_solder, marbastlib-mx:SW_MX_1u, F.Cu at (130.7, 94.1)
- added SW42: MX_SW_solder, marbastlib-mx:SW_MX_1u, F.Cu at (152.1, 94.1)
- added SW43: ROT_SKYLOONG_HS, PCM_marbastlib-various:ROT_SKYLOONG_HS-Switch, F.Cu at (47.3, 36.9)
- added SW44: ROT_SKYLOONG_HS, PCM_marbastlib-various:ROT_SKYLOONG_HS-Switch, F.Cu at (256.9, 36.9)
- added SW45: MX_SW_solder, marbastlib-mx:SW_MX_1u, F.Cu at (178.3, 94.1)
- added SW46: MX_SW_solder, marbastlib-mx:SW_MX_1u, F.Cu at (180.7, 94.1)
- added SW47: MX_SW_solder, marbastlib-mx:SW_MX_1u, F.Cu at (209.2, 94.1)
- added SW48: MX_SW_solder, marbastlib-mx:SW_MX_1u, F.Cu at (237.8, 94.1)
- added SW49: MX_SW_solder, marbastlib-mx:SW_MX_1.5u, F.Cu at (233.0, 94.1)
- added SW5: MX_SW_solder, marbastlib-mx:SW_MX_1u, F.Cu at (123.5, 36.9)
- added SW50: MX_SW_solder, marbastlib-mx:SW_MX_1u, F.Cu at (218.8, 94.1)
- added SW51: MX_SW_solder, marbastlib-mx:SW_MX_1u, F.Cu at (256.9, 94.1)
- added SW52: MX_SW_solder, marbastlib-mx:SW_MX_1u, F.Cu at (245.0, 75.0)
- added SW53: SW_Push, Button_Switch_SMD:SW_SPST_SKQG_WithoutStem, B.Cu at (19.1, 42.8)
- added SW6: MX_SW_solder, marbastlib-mx:SW_MX_1u, F.Cu at (142.6, 36.9)
- added SW7: MX_SW_solder, marbastlib-mx:SW_MX_1u, F.Cu at (161.6, 36.9)
- added SW8: MX_SW_solder, marbastlib-mx:SW_MX_1u, F.Cu at (180.7, 36.9)
- added SW9: MX_SW_solder, marbastlib-mx:SW_MX_1u, F.Cu at (199.7, 36.9)
- added U6: STM32L443CCUx, Package_DFN_QFN:QFN-48-1EP_7x7mm_P0.5mm_EP5.6x5.6mm, B.Cu at (67.5, 69.1)
- D1, D2, D3, D4: moved to B.Cu
- J1: value USB_C_Receptacle_USB2.0 -> Conn_01x04_MountingPin; footprint Connector_USB:USB_C_Receptacle_GCT_USB4085 -> Connector_Molex:Molex_Pico-EZmate_78171-0004_1x04-1MP_P1.20mm_Vertical; moved to B.Cu
- R5: value 5.1k -> 100k; moved to B.Cu
- U2: value SOP-8 SPI FLASH -> 3.3V Fixed Regulator; footprint Package_SO:SOP-8_3.76x4.96mm_P1.27mm -> Package_TO_SOT_SMD:TSOT-23; moved to B.Cu
- moved SW4 87.2 mm to (104.5, 36.9)
- moved R5 70.8 mm to (40.8, 39.4), turned to 180 degrees
- moved SW3 59.5 mm to (85.4, 36.9)
- moved D1 46.6 mm to (47.3, 41.7)
- moved D4 46.1 mm to (104.5, 41.7)
- moved D2 37.6 mm to (66.4, 41.7)
- moved D3 37.3 mm to (85.4, 41.7)
- moved SW2 31.7 mm to (66.4, 36.9)
- moved J1 31.5 mm to (75.9, 44.1), turned to -90 degrees
- moved U2 20.5 mm to (60.2, 46.4)
- moved SW1 4.03 mm to (47.3, 36.9)
Connections:
- net Net-(D1-A) renamed /Switch Matrix/SKY_MAT_1
- D1 pad 1: GP0 -> GP26
- D2 pad 1: GP0 -> GP26
- D3 pad 1: GP1 -> GP26
- D4 pad 1: GP1 -> GP26
- R5 pad 1: GND -> Net-(Q3-G)
- R5 pad 2: Net-(J1-CC2) -> +3.3V
- SW1 pad 1: GP2 -> GP1
- SW2 pad 1: GP3 -> GP0
- SW3 pad 1: GP2 -> GP21
- SW4 pad 1: GP3 -> GP28
- U2 pad 1: /CS_ -> GND
- U2 pad 2: /SD1_ -> +3.3V
- U2 pad 3: /SD2_ -> /VFused_
Routing:
- added copper zone on In2.Cu, net +3.3V
- added copper zone on B.Cu, net GND
- added copper zone on F.Cu, net GND
- added copper zone on In1.Cu, net GND
Other:
- board outline added: 227.1 x 74.7 mm
