File: PCB.kicad_sch (KiCad schematic)
At the start: 34 parts, among them J1 USB_C_Receptacle_USB2.0, J2 JST - 1.00mm 4 Pin, SW72 SW_Push, SW73 SW_Push, U1 RP2040, U2 SOP-8 SPI FLASH, U3 USBLC6-2SC6, U4 3.3V Fixed Regulator, Y1 12MHz Crystal 3225

Commit message: Layout complete
Parts:
- removed C1, C2: 30p, Capacitor_SMD:C_0402_1005Metric, symbol Device:C_Small
- removed C10, C12, C13, C15, C3: 1u, Capacitor_SMD:C_0402_1005Metric, symbol Device:C_Small
- removed C11, C14, C16, C4, C5, C6, C7, C8, C9: 100n, Capacitor_SMD:C_0402_1005Metric, symbol Device:C_Small
- removed D65: LED, marbastlib-mx:LED_MX_3mm, symbol Device:LED
- removed F1: 700mA, Fuse:Fuse_0402_1005Metric, symbol Device:Polyfuse_Small
- removed FB1: 100 Ohm @ 100 MHz, Inductor_SMD:L_0402_1005Metric, symbol Device:FerriteBead_Small
- removed J1: USB_C_Receptacle_USB2.0, Connector_USB:USB_C_Receptacle_GCT_USB4085, symbol Connector:USB_C_Receptacle_USB2.0
- removed J2: JST - 1.00mm 4 Pin, Connector_JST:JST_SH_SM04B-SRSS-TB_1x04-1MP_P1.00mm_Horizontal, symbol Connector_Generic_MountingPin:Conn_01x04_MountingPin
- removed R1, R2: 22, Resistor_SMD:R_0402_1005Metric, symbol Device:R_Small_US
- removed R3: 1k, Resistor_SMD:R_0402_1005Metric, symbol Device:R_Small_US
- removed R4, R5: 5.1k, Resistor_SMD:R_0402_1005Metric, symbol Device:R_Small_US
- removed R7: R_Small_US, Resistor_SMD:R_0402_1005Metric, symbol Device:R_Small_US
- removed SW72, SW73: SW_Push, Button_Switch_SMD:SW_SPST_SKQG_WithoutStem, symbol Switch:SW_Push
- removed U1: RP2040, Package_DFN_QFN:QFN-56-1EP_7x7mm_P0.4mm_EP3.2x3.2mm_ThermalVias, symbol MCU_RaspberryPi:RP2040
- removed U2: SOP-8 SPI FLASH, Package_SO:SOP-8_3.76x4.96mm_P1.27mm, symbol Memory_Flash:MX25R3235FZNxx0
- removed U3: USBLC6-2SC6, Package_TO_SOT_SMD:SOT-23-6, symbol Power_Protection:USBLC6-2SC6
- removed U4: 3.3V Fixed Regulator, Package_TO_SOT_SMD:TSOT-23, symbol Regulator_Linear:AP2127N3-1.2
- removed Y1: 12MHz Crystal 3225, Crystal:Crystal_SMD_3225-4Pin_3.2x2.5mm, symbol Device:Crystal_GND24_Small
- added C17, C18: 1u, Capacitor_SMD:C_0402_1005Metric, symbol Device:C_Small
- added C19: 4.7u, Capacitor_SMD:C_0402_1005Metric, symbol Device:C_Small
- added C20, C21, C22, C23: 100n, Capacitor_SMD:C_0402_1005Metric, symbol Device:C_Small
- added D45: LED, Resistor_SMD:R_0603_1608Metric, symbol Device:LED
- added J3: Conn_01x04_MountingPin, Connector_Molex:Molex_Pico-EZmate_78171-0004_1x04-1MP_P1.20mm_Vertical, symbol Connector_Generic_MountingPin:Conn_01x04_MountingPin
- added J4: TC2030_SWD, PCM_marbastlib-various:CON_TC2030_outlined, symbol PCM_marbastlib-various:TC2030_SWD
- added Q4: PMOS, Package_TO_SOT_SMD:SOT-323_SC-70, symbol Device:Q_PMOS_GSD
- added R8: 470, Resistor_SMD:R_0603_1608Metric, symbol Device:R_Small_US
- added SW53: SW_Push, Button_Switch_SMD:SW_SPST_SKQG_WithoutStem, symbol Switch:SW_Push
- added U2: 3.3V Fixed Regulator, Package_TO_SOT_SMD:TSOT-23, symbol Regulator_Linear:AP2127N3-1.2
- added U6: STM32L443CCUx, Package_DFN_QFN:QFN-48-1EP_7x7mm_P0.5mm_EP5.6x5.6mm, symbol MCU_ST_STM32L4:STM32L443CCUx
Connections:
- net +3.3V: now also C18.1, C19.1, C20.1, C21.1, C22.1, C23.1, J4.1 (VCC), U2.2 (VO), U6.24 (VDD), U6.36 (VDDUSB), U6.48 (VDD), U6.9 (VDDA)
- net DN: now also J3.3 (Pin_3), U6.32 (PA11)
- net DP: now also J3.2 (Pin_2), U6.33 (PA12)
- net GND: now also C17.2, C18.2, C19.2, C20.2, C21.2, C22.2, C23.2, J3.1 (Pin_1), J3.MP (MountPin), J4.5 (GND), Q4.1 (G), R8.1, SW53.1, U2.1 (GND), U6.23 (VSS), U6.35 (VSS), U6.47 (VSS), U6.49 (VSS), U6.8 (VSSA)
- net RUN_: now also J4.3 (~{RST})
- net VFused_: now also C17.1, Q4.2 (S), U2.3 (VI)
- new net: D45.2 (A), R8.2
- new net: D45.1 (K), J3.4 (Pin_4), Q4.3 (D)
- new net SWCLK: J4.4 (SWCLK)
- new net SWD: J4.6 (SWO)
- new net ~{RST}: SW53.2, U6.7 (NRST)
- no-connect marks 3 -> 2
Other:
- note removed: "C1, C2 = 2*CL - 2*5pF Where CL, or load capacitance, is given by your crystal's datasheet."
- note removed: "Crystal"
- note removed: "Flash Memory"
- note removed: "Indicator LED"
