File: switch_matrix.kicad_sch (KiCad schematic)
At the start: 8 parts, among them SW1 MX_SW_solder, SW2 MX_SW_solder, SW3 MX_SW_solder, SW4 MX_SW_solder

Commit message: Layout complete
Parts:
- removed SW2, SW3, SW4: MX_SW_solder, marbastlib-mx:SW_MX_1u, symbol marbastlib-mx:MX_SW_solder
- added D10, D11, D12, D13, D14, D15, D16, D17, D18, D19, D20, D21, D22, D23, D24, D25, D26, D27, D28, D29, D30, D31, D32, D33, D34, D35, D36, D37, D38, D39, D40, D41, D42, D44, D5, D6, D7, D8, D9: D_Small, Diode_SMD:D_SOD-123, symbol Device:D_Small
- added Q1 (x2): PMOS, Package_TO_SOT_SMD:SOT-323_SC-70, symbol Device:Q_PMOS_GSD
- added R3 (x2): 100k, Resistor_SMD:R_0402_1005Metric, symbol Device:R_Small_US
- added S1: MX_stab, marbastlib-mx:STAB_MX_P_7u, symbol marbastlib-mx:MX_stab
- added S2: MX_stab, marbastlib-mx:STAB_MX_P_10u, symbol marbastlib-mx:MX_stab
- added S3, S40: MX_stab, marbastlib-mx:STAB_MX_P_3u, symbol marbastlib-mx:MX_stab
- added S35, S4: MX_stab, marbastlib-mx:STAB_MX_P_2.25u, symbol marbastlib-mx:MX_stab
- added S41: MX_stab, marbastlib-mx:STAB_MX_P_2.75u, symbol marbastlib-mx:MX_stab
- added SW10, SW11, SW12, SW14, SW15, SW16, SW17, SW18, SW19, SW2, SW20, SW21, SW22, SW25, SW26, SW27, SW28, SW29, SW3, SW30, SW31, SW32, SW33, SW35, SW36, SW38, SW39, SW4, SW40, SW41, SW42, SW45, SW46, SW47, SW48, SW5, SW50, SW51, SW52, SW6, SW7, SW8, SW9: MX_SW_solder, marbastlib-mx:SW_MX_1u, symbol marbastlib-mx:MX_SW_HS
- added SW13, SW34: MX_SW_solder, marbastlib-mx:SW_MX_1.25u, symbol marbastlib-mx:MX_SW_HS
- added SW23, SW24: MX_SW_solder, marbastlib-mx:SW_MX_1.75u, symbol marbastlib-mx:MX_SW_HS
- added SW37, SW49: MX_SW_solder, marbastlib-mx:SW_MX_1.5u, symbol marbastlib-mx:MX_SW_HS
- added SW43, SW44: ROT_SKYLOONG_HS, PCM_marbastlib-various:ROT_SKYLOONG_HS-Switch, symbol PCM_marbastlib-various:ROT_SKYLOONG_HS-Switch
- SW1: symbol marbastlib-mx:MX_SW_solder -> marbastlib-mx:MX_SW_HS
Connections:
- net GP0: now also SW14.1, SW2.1, SW25.1, SW36.1, SW37.1; no longer D1.1 (K), D2.1 (K)
- net GP1: now also SW1.1, SW13.1, SW24.1, SW35.1; no longer D3.1 (K), D4.1 (K)
- net GP2: now also SW18.1, SW29.1, SW42.1, SW6.1; no longer SW1.1
- net GP21: now also SW15.1, SW26.1, SW3.1, SW38.1, SW39.1
- net GP23: now also SW17.1, SW28.1, SW5.1
- net GP24: now also D24.1 (K), D25.1 (K), D26.1 (K), D27.1 (K), D28.1 (K), D29.1 (K), D30.1 (K), D31.1 (K), D32.1 (K), D33.1 (K), D34.1 (K)
- net GP25: now also D35.1 (K), D36.1 (K), D37.1 (K), D38.1 (K), D39.1 (K), D40.1 (K), D41.1 (K), D42.1 (K), D44.1 (K)
- net GP26: now also D1.1 (K), D2.1 (K), D3.1 (K), D4.1 (K), D10.1 (K), D11.1 (K), D12.1 (K), D5.1 (K), D6.1 (K), D7.1 (K), D8.1 (K), D9.1 (K), Q1.3 (D), Q1.3 (D)
- net GP27: now also D13.1 (K), D14.1 (K), D15.1 (K), D16.1 (K), D17.1 (K), D18.1 (K), D19.1 (K), D20.1 (K), D21.1 (K), D22.1 (K), D23.1 (K)
- net GP28: now also SW16.1, SW27.1, SW4.1, SW40.1, SW41.1
- net GP3: now also SW19.1, SW30.1, SW45.1, SW46.1, SW7.1
- net GP4: now also SW20.1, SW31.1, SW47.1, SW48.1, SW8.1
- net GP5: now also SW21.1, SW32.1, SW49.1, SW50.1, SW9.1
- net GP6: now also SW10.1, SW22.1, SW33.1
- net GP8: now also SW11.1, SW23.1, SW34.1, SW51.1, SW52.1
- net GP9: now also SW12.1
- net at D2.2 (A): now also SW2.2
- net SKY_MAT_1: now reaches D1.2 (A), SW1.2
- net SKY_MAT_1: now also Q1.2 (S)
- net at D3.2 (A): now also SW3.2
- net at D4.2 (A): now also SW4.2
- new net: D36.2 (A), SW36.2
- new net: D29.2 (A), SW29.2
- new net: Q1.1 (G), R3.1, SW44.S
- new net: D35.2 (A), SW35.2
- new net: D9.2 (A), SW9.2
- new net: D5.2 (A), SW5.2
- new net: D10.2 (A), SW10.2
- new net: D17.2 (A), SW17.2
- new net: D15.2 (A), SW15.2
- new net: D42.2 (A), SW50.2
- new net: D38.2 (A), SW40.2
- new net: D27.2 (A), SW27.2
- new net: D23.2 (A), SW23.2
- new net: D26.2 (A), SW26.2
- new net: D31.2 (A), SW31.2
- new net: D34.2 (A), SW34.2, SW52.2
- new net: D19.2 (A), SW19.2
- new net: D13.2 (A), SW13.2
- new net: D41.2 (A), SW45.2
- new net: D22.2 (A), SW22.2
- new net: D25.2 (A), SW25.2
- new net: D14.2 (A), SW14.2
- new net: D21.2 (A), SW21.2
- new net: Q1.1 (G), R3.1, SW43.S
- new net: D39.2 (A), SW47.2
- new net: D20.2 (A), SW20.2
- new net: D33.2 (A), SW33.2
- new net: D18.2 (A), SW18.2
- new net: D44.2 (A), SW51.2
- new net: D7.2 (A), SW7.2
- new net: D8.2 (A), SW8.2
- new net: D11.2 (A), SW11.2
- new net: D28.2 (A), SW28.2
- new net: D6.2 (A), SW6.2
- new net: D32.2 (A), SW32.2
- new net: D40.2 (A), SW42.2
- new net: D37.2 (A), SW38.2
- new net: D24.2 (A), SW24.2
- new net: D16.2 (A), SW16.2
- new net: D30.2 (A), SW30.2
- new net +3.3V: R3.2, R3.2
- new net GND: SW43.C, SW44.C
- new net SKY_MAT_2: D12.2 (A), Q1.2 (S), SW12.2
Other:
- moved on the sheet: D1, SW1

Commit message: Stagger
Connections:
- net at D36.2 (A), SW36.2: now also SW37.2
- net at SW46.2: now also D41.2 (A), SW45.2
- net ENC1A: now reaches SW44.A
- net ENC1B: now reaches SW44.B
- net at SW50.2: now also D39.2 (A), SW47.2; no longer D42.2 (A)
- net at D38.2 (A), SW40.2: now also SW41.2
- net at SW39.2: now also D37.2 (A), SW38.2
- net at SW49.2: now also D42.2 (A), SW48.2
- net ENC0A: now reaches SW43.A
- net ENC0B: now reaches SW43.B
- net GP0 renamed COL1
- net GP1 renamed COL0
- net COL0: now also Q1.2 (S)
- net GP2 renamed COL5
- net GP21 renamed COL2
- net GP23 renamed COL4
- net GP24 renamed ROW2
- net GP25 renamed ROW3
- net GP26 renamed ROW0
- net ROW0: no longer Q1.3 (D), Q1.3 (D)
- net GP27 renamed ROW1
- net GP28 renamed COL3
- net GP3 renamed COL6
- net GP4 renamed COL7
- net COL7: now also SW50.1; no longer SW48.1
- net GP5 renamed COL8
- net COL8: now also SW48.1; no longer SW50.1
- net GP6 renamed COL9
- net GP8 renamed COL10
- net GP9 renamed COL11
- net COL11: now also Q1.2 (S)
- net SKY_MAT_1 renamed D1
- net D1: now also Q1.3 (D); no longer Q1.2 (S)
- net SKY_MAT_2 renamed D12
- net D12: now also Q1.3 (D); no longer Q1.2 (S)
